Commit message: Added robot model sdf and urdf but with some issues to fix for the sdf

File: orto_nav/urdf/sam_bot_description.urdf (robot description, URDF)
Before this commit: robot sam_bot, 7 links, 6 joints
Links:
- removed link imu_link
Joints:
- removed joint imu_joint
- joint base_joint: child base_footprint -> base_link; parent base_link -> base_footprint
- joint laser_joint: origin xyz=0.16  0    0.12 rpy=0  0  0 -> xyz=0.16 0 0.12 rpy=0  0  0

Commit message: Fixed nav2 issues

File: orto_nav/urdf/sam_bot_description.urdf (robot description, URDF)
Before this commit: robot orthopillar, 6 links, 5 joints
Joints:
- joint drivewhl_l_joint: limit (none) -> effort=10000 velocity=1000; type continuous -> revolute
- joint drivewhl_r_joint: limit (none) -> effort=10000 velocity=1000; type continuous -> revolute

File: sam_bot_description/src/description/sam_bot_description.urdf (robot description, URDF)
Before this commit: robot sam_bot, 5 links, 4 joints
Links:
- removed link base_footprint
Joints:
- removed joint base_joint
